File: 2_prototype_mk1/hardware/sdcard_reader.kicad_sch (KiCad schematic)
At the start: 4 parts, among them J1 Micro_SD_Card

Commit message: Switch out SD card reader for correct footprint
Parts:
- J1: footprint Connector_Card:microSD_HC_Hirose_DM3AT-SF-PEJM5 -> Connector_Card:microSD_HC_Hirose_DM3D-SF
Connections:
- net SD_CS: now also RN2.1 (R1.1); no longer RN2.3 (R3.1)
- net SD_MISO: now also RN2.3 (R3.1); no longer RN2.1 (R1.1)
Other:
- note added: "Hirose DM3D-SF Manual push/pull Ideal for internal use"
Changed lines of the file:
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@@
+		)
+	)
+	(text "Hirose DM3D-SF\nManual push/pull \nIdeal for internal use"
+		(exclude_from_sim no)
+		(at 127.762 68.834 0)
+		(effects
+			(font
+				(size 1.27 1.27)
+			)
+			(justify left)
 		)
 	)
@@
 	)
 	(junction
-		(at 88.9 87.63)
+		(at 88.9 92.71)
+		(diameter 0)
+		(color 0 0 0 0)
+	)
+	(junction
+		(at 83.82 87.63)
 		(diameter 0)
 		(color 0 0 0 0)
@@
 	)
 	(junction
-		(at 83.82 92.71)
-		(diameter 0)
-		(color 0 0 0 0)
-	)
-	(junction
 		(at 86.36 71.12)
 		(diameter 0)
@@
 	(wire
 		(pts
+			(xy 83.82 87.63) (xy 124.46 87.63)
+		)
+		(stroke
+			(width 0)
+			(type default)
+		)
+	)
+	(wire
+		(pts
 			(xy 107.95 113.03) (xy 107.95 114.3)
 		)
@@
 	(wire
 		(pts
+			(xy 83.82 82.55) (xy 83.82 87.63)
+		)
+		(stroke
+			(width 0)
+			(type default)
+		)
+	)
+	(wire
+		(pts
 			(xy 96.52 92.71) (xy 96.52 100.33)
 		)
@@
 	(wire
 		(pts
-			(xy 83.82 82.55) (xy 83.82 92.71)
+			(xy 88.9 92.71) (xy 96.52 92.71)
 		)
 		(stroke
@@
 	(wire
 		(pts
-			(xy 77.47 92.71) (xy 83.82 92.71)
+			(xy 77.47 92.71) (xy 88.9 92.71)
 		)
 		(stroke
@@
 	(wire
 		(pts
-			(xy 88.9 82.55) (xy 88.9 87.63)
-		)
-		(stroke
-			(width 0)
-			(type default)
-		)
-	)
-	(wire
-		(pts
 			(xy 167.64 107.95) (xy 167.64 113.03)
 		)
@@
 	(wire
 		(pts
-			(xy 77.47 87.63) (xy 88.9 87.63)
-		)
-		(stroke
-			(width 0)
-			(type default)
-		)
-	)
-	(wire
-		(pts
-			(xy 83.82 92.71) (xy 96.52 92.71)
+			(xy 77.47 87.63) (xy 83.82 87.63)
 		)
 		(stroke
@@
 	(wire
 		(pts
-			(xy 88.9 87.63) (xy 124.46 87.63)
+			(xy 88.9 82.55) (xy 88.9 92.71)
 		)
 		(stroke
@@
 			)
 		)
-		(property "Footprint" "Connector_Card:microSD_HC_Hirose_DM3AT-SF-PEJM5"
+		(property "Footprint" "Connector_Card:microSD_HC_Hirose_DM3D-SF"
 			(at 176.53 85.09 0)
 			(hide yes)
@@
 			)
 		)
-		(property "Description" "Micro SD Card Socket"
+		(property "Description" "Micro SD Card Socket - Hirose DM3D-SF"
 			(at 147.32 92.71 0)
 			(hide yes)
