File: 2_prototype_mk1/hardware/power.kicad_sch (KiCad schematic)
At the start: 2 parts, among them J4 Conn_01x04_Pin

Commit message: Change power connector and reroute amp
Parts:
- J4: footprint Connector_JST:JST_XH_B4B-XH-A_1x04_P2.50mm_Vertical -> Connector_Molex:Molex_KK-254_AE-6410-04A_1x04_P2.54mm_Vertical
Changed lines of the file:
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@@
 			)
 		)
-		(property "Footprint" "Connector_JST:JST_XH_B4B-XH-A_1x04_P2.50mm_Vertical"
+		(property "Footprint" "Connector_Molex:Molex_KK-254_AE-6410-04A_1x04_P2.54mm_Vertical"
 			(at 130.81 104.14 0)
 			(hide yes)
